File: rs-probe.kicad_sch (KiCad schematic)
At the start: 98 parts, among them J1 USB_C_Receptacle_USB2.0, J10 Conn_01x01, J11 Conn_01x01, J2 Castellated Vias, J3 Castellated Vias, J4 Castellated Vias, J5 tag-connect-swd, J6 Conn_01x01, J7 Conn_01x01, J8 Conn_01x01, J9 Conn_01x01, Q1 NTZD3155C or CMLDM3757-TR-PBF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, SW1 EVQ-P2002W, T1 Tab, T2 Tab, U1 74LVC1T45GM,115, U10 74LVC1T45GM,115, U11 74LVC1T45GM,115, U12 NCP133AMXADJTCG, U13 NCP133AMXADJTCG, U14 NCP133AMXADJTCG, U2 74LVC1T45GM,115, U3 W25Q8, U4 NUF8401MNT4G, U5 CortexDebug, U6 RP2040, U7 NUF2042XV6T1G, U8 74LVC1T45GM,115, U9 74LVC1T45GM,115, X1 12 MHz

Commit message: Lots of work
Parts:
- removed J10, J11: Conn_01x01, connectors:pad_1.5x2.0mm, symbol Connector_Generic:Conn_01x01
- removed J2: Castellated Vias, connectors:1x9_1.5mm_castellated, symbol Connector_Generic:Conn_01x09
- removed J3: Castellated Vias, connectors:1x2_1.5mm_castellated, symbol Connector_Generic:Conn_01x02
- removed J4: Castellated Vias, connectors:1x3_1.5mm_castellated, symbol Connector_Generic:Conn_01x03
- removed TP1, TP2, TP3, TP4: TestPoint, TestPoint:TestPoint_Pad_D1.0mm, symbol Connector:TestPoint
- added C31, C32, C33, C34, C35: 0.1u, passive:C_0402, symbol Device:C_Small
- added J1, J2, J3, J5: Conn_01x01, connectors:pad_2.0x2.5mm, symbol Connector_Generic:Conn_01x01
- J6, J7, J8, J9: footprint connectors:pad_1.5x2.0mm -> connectors:pad_2.0x2.5mm; now in the parts list
- R10, R18, R22, R23, R24, R26: value 1Meg -> 1M
- X1: renamed from U5; value CortexDebug -> Conn_ST_STDC14; symbol connectors:Cortex-Debug -> Connector:Conn_ARM_JTAG_SWD_10; LCSC C2935458, C150517, C920815 -> C448647
- X10: renamed from J1; symbol Connector:USB_C_Receptacle_USB2.0 -> Connector:USB_C_Receptacle_USB2.0_16P
- X5: renamed from J5; value tag-connect-swd -> TagConnect; symbol connectors:tag-connect-swd -> Connector:Conn_ARM_SWD_TagConnect_TC2030-NL
- renumbered X1 to XC1
Connections:
- net +3.3V: now also C34.1, C35.1
- net 5V_KEY: now also J6.1 (Pin_1); no longer X1.7 (T_JRCLK)
- net GND: now also C31.2, C32.2, C33.2, C34.2, C35.2, J1.1 (Pin_1), J5.1 (Pin_1); no longer J6.1 (Pin_1)
- net GPIO1: now also J9.1 (Pin_1)
- net GPIO2: now also J7.1 (Pin_1)
- net TRANS_VCC: now also C31.1, C32.1, C33.1
- net T_SWDCLK_JCLK: no longer J9.1 (Pin_1)
- net T_SWDIO_TMS: no longer J8.1 (Pin_1)
- net T_VCC: now also J8.1 (Pin_1); no longer J7.1 (Pin_1)
- net T_VCP_RX: now also J3.1 (Pin_1)
- net T_VCP_TX: now also J2.1 (Pin_1)
Other:
- note added: "0.5A hold 1A trip"
- note removed: "0.5A hold, 1A trip"
- moved on the sheet: R16, R2, R27, SW1, U4

Commit message: wip
Parts:
- SW1: footprint Button_Switch_SMD:SW_SPST_EVQP2 -> pushbuttons:PCB_JumperButton
Changed lines of the file:
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@@
 			)
 		)
-		(property "Footprint" "Button_Switch_SMD:SW_SPST_EVQP2"
+		(property "Footprint" "pushbuttons:PCB_JumperButton"
 			(at 31.75 143.51 0)
 			(effects

Commit message: wip
Connections:
- net DIR_SWDCLK_JCLK: now also U6.16 (GPIO13); no longer U6.30 (GPIO19)
- net DIR_TDI: now also U6.29 (GPIO18); no longer U6.35 (GPIO23)
- net DIR_VCP_TX: now also U6.30 (GPIO19); no longer U6.36 (GPIO24)
- net GNDDetect: now also U6.17 (GPIO14); no longer U6.11 (GPIO8)
- net ~{RESET}: now also U6.18 (GPIO15); no longer U6.12 (GPIO9)
Other:
- note added: "DESIGN NOTE: T_VCC is read before enabling power."
- note removed: "DESIGN NOTE: T_VCC is read before enabling ower."
Changed lines of the file:
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@@
 	)
 	(no_connect
-		(at 109.22 107.95)
+		(at 121.92 220.98)
 	)
 	(no_connect
-		(at 58.42 200.66)
+		(at 121.92 180.34)
 	)
 	(no_connect
-		(at 226.06 259.08)
+		(at 121.92 182.88)
 	)
 	(no_connect
-		(at 121.92 170.18)
+		(at 109.22 107.95)
 	)
 	(no_connect
-		(at 121.92 198.12)
+		(at 58.42 200.66)
 	)
 	(no_connect
-		(at 121.92 205.74)
+		(at 121.92 218.44)
 	)
 	(no_connect
-		(at 121.92 193.04)
+		(at 226.06 259.08)
 	)
 	(no_connect
-		(at 121.92 195.58)
+		(at 121.92 170.18)
 	)
 	(no_connect
@@
 		)
 	)
-	(text "DESIGN NOTE:\nT_VCC is read before \nenabling ower."
+	(text "DESIGN NOTE:\nT_VCC is read before \nenabling power."
 		(exclude_from_sim no)
 		(at 212.09 35.56 0)
@@
 		)
 	)
+	(global_label "DIR_TDI"
+		(shape input)
+		(at 121.92 205.74 0)
+		(fields_autoplaced yes)
+		(effects
+			(font
+				(size 1.27 1.27)
+			)
+			(justify left)
+		)
+		(property "Intersheetrefs" "${INTERSHEET_REFS}"
+			(at 131.86 205.74 0)
+			(effects
+				(font
+					(size 1.27 1.27)
+				)
+				(justify left)
+				(hide yes)
+			)
+		)
+	)
 	(global_label "PWM_VS"
 		(shape input)
@@
 		)
 	)
+	(global_label "DIR_VCP_TX"
+		(shape input)
+		(at 121.92 208.28 0)
+		(fields_autoplaced yes)
+		(effects
+			(font
+				(size 1.27 1.27)
+			)
+			(justify left)
+		)
+		(property "Intersheetrefs" "${INTERSHEET_REFS}"
+			(at 135.7909 208.28 0)
+			(effects
+				(font
+					(size 1.27 1.27)
+				)
+				(justify left)
+				(hide yes)
+			)
+		)
+	)
 	(global_label "T_SWDCLK_JCLK"
 		(shape input)
@@
 		)
 	)
+	(global_label "DIR_SWO_TDO"
+		(shape input)
+		(at 121.92 215.9 0)
+		(fields_autoplaced yes)
+		(effects
+			(font
+				(size 1.27 1.27)
+			)
+			(justify left)
+		)
+		(property "Intersheetrefs" "${INTERSHEET_REFS}"
+			(at 137.5447 215.9 0)
+			(effects
+				(font
+					(size 1.27 1.27)
+				)
+				(justify left)
+				(hide yes)
+			)
+		)
+	)
 	(global_label "P_SWCLK"
 		(shape input)
@@
 		)
 	)
-	(global_label "DIR_SWDCLK_JCLK"
-		(shape input)
-		(at 121.92 208.28 0)
-		(fields_autoplaced yes)
-		(effects
-			(font
-				(size 1.27 1.27)
-			)
-			(justify left)
-		)
-		(property "Intersheetrefs" "${INTERSHEET_REFS}"
-			(at 142.0199 208.28 0)
-			(effects
-				(font
-					(size 1.27 1.27)
-				)
-				(justify left)
-				(hide yes)
-			)
-		)
-	)
 	(global_label "TRANS_VCC"
 		(shape input)
@@
 	(global_label "~{RESET}"
 		(shape input)
-		(at 121.92 182.88 0)
+		(at 121.92 198.12 0)
 		(fields_autoplaced yes)
 		(effects
@@
 		)
 		(property "Intersheetrefs" "${INTERSHEET_REFS}"
-			(at 130.6503 182.88 0)
+			(at 130.6503 198.12 0)
 			(effects
 				(font
@@
 		)
 	)
-	(global_label "DIR_VCP_TX"
-		(shape input)
-		(at 121.92 220.98 0)
-		(fields_autoplaced yes)
-		(effects
-			(font
-				(size 1.27 1.27)
-			)
-			(justify left)
-		)
-		(property "Intersheetrefs" "${INTERSHEET_REFS}"
-			(at 135.7909 220.98 0)
-			(effects
-				(font
-					(size 1.27 1.27)
-				)
-				(justify left)
-				(hide yes)
-			)
-		)
-	)
 	(global_label "5V_KEY_EN"
 		(shape input)
@@
 		)
 	)
-	(global_label "GNDDetect"
-		(shape input)
-		(at 121.92 180.34 0)
-		(fields_autoplaced yes)
-		(effects
-			(font
-				(size 1.27 1.27)
-			)
-			(justify left)
-		)
-		(property "Intersheetrefs" "${INTERSHEET_REFS}"
-			(at 134.7629 180.34 0)
-			(effects
-				(font
-					(size 1.27 1.27)
-				)
-				(justify left)
-				(hide yes)
-			)
-		)
-	)
 	(global_label "T_~{RESET}"
 		(shape input)
@@
 		)
 	)
-	(global_label "D_FS_N"
+	(global_label "DIR_SWDCLK_JCLK"
 		(shape input)
-		(at 180.34 245.11 180)
+		(at 121.92 193.04 0)
 		(fields_autoplaced yes)
 		(effects
@@
 				(size 1.27 1.27)
 			)
-			(justify right)
+			(justify left)
 		)
 		(property "Intersheetrefs" "${INTERSHEET_REFS}"
-			(at 170.521 245.11 0)
+			(at 142.0199 193.04 0)
 			(effects
 				(font
 					(size 1.27 1.27)
 				)
-				(justify right)
+				(justify left)
 				(hide yes)
 			)
 		)
 	)
-	(global_label "T_SWO_TDO"
+	(global_label "GNDDetect"
 		(shape input)
-		(at 213.36 76.2 0)
+		(at 121.92 195.58 0)
 		(fields_autoplaced yes)
 		(effects
@@
 		)
 		(property "Intersheetrefs" "${INTERSHEET_REFS}"
-			(at 226.8075 76.2 0)
+			(at 134.7629 195.58 0)
 			(effects
 				(font
@@
 		)
 	)
-	(global_label "DIR_SWO_TDO"
+	(global_label "D_FS_N"
 		(shape input)
-		(at 121.92 215.9 0)
+		(at 180.34 245.11 180)
+		(fields_autoplaced yes)
+		(effects
+			(font
+				(size 1.27 1.27)
+			)
+			(justify right)
+		)
+		(property "Intersheetrefs" "${INTERSHEET_REFS}"
+			(at 170.521 245.11 0)
+			(effects
+				(font
+					(size 1.27 1.27)
+				)
+				(justify right)
+				(hide yes)
+			)
+		)
+	)
+	(global_label "T_SWO_TDO"
+		(shape input)
+		(at 213.36 76.2 0)
 		(fields_autoplaced yes)
 		(effects
@@
 		)
 		(property "Intersheetrefs" "${INTERSHEET_REFS}"
-			(at 137.5447 215.9 0)
+			(at 226.8075 76.2 0)
 			(effects
 				(font
@@
 				(hide yes)
 			)
-		)
-	)
-	(global_label "DIR_TDI"
-		(shape input)
-		(at 121.92 218.44 0)
-		(fields_autoplaced yes)
-		(effects
-			(font
-				(size 1.27 1.27)
-			)
-			(justify left)
-		)
-		(property "Intersheetrefs" "${INTERSHEET_REFS}"
-			(at 131.86 218.44 0)
-			(effects
-				(font
-					(size 1.27 1.27)
-				)
-				(justify left)
-				(hide yes)
-			)

Commit message: clearing drc errors
Parts:
- U14: footprint Package_DFN_QFN:DFN-6-1EP_1.2x1.2mm_P0.4mm_EP0.3x0.94mm_PullBack -> dfn:DFN-6-1EP_1.2x1.2mm_P0.4mm_EP0.3x0.94mm_PullBack
Changed lines of the file:
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@@
 			)
 		)
-		(property "Footprint" "Package_DFN_QFN:DFN-6-1EP_1.2x1.2mm_P0.4mm_EP0.3x0.94mm_PullBack"
+		(property "Footprint" "dfn:DFN-6-1EP_1.2x1.2mm_P0.4mm_EP0.3x0.94mm_PullBack"
 			(at 241.3 132.08 0)
 			(effects

Commit message: fixing missing 3D models
Parts:
- D2: LCSC (none) -> C2837790; MFPN SBA0520Q or similar -> RB161QS-40T18R
- D3: LCSC (none) -> C2837790; MFPN SBA0520Q or similar -> RB161QS-40T18R; Rectified Current (none) -> 500mA; VfVr (none) -> 20V
- FB1: LCSC (none) -> C76886
- J1, J2, J3, J5, J6, J7, J8, J9: now left out of the parts list
- U1, U10, U11, U2, U8, U9: value 74LVC1T45GM,115 -> 74LVC1T45GM-Q100X; LCSC C548481, C548480, C548479 -> C548481; MFPN 74LVC1T45GM,115 -> 74LVC1T45GM-Q100X
Changed lines of the file:
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@@
 		(unit 1)
 		(exclude_from_sim no)
-		(in_bom yes)
+		(in_bom no)
 		(on_board yes)
 		(dnp no)
@@
 		(unit 1)
 		(exclude_from_sim no)
-		(in_bom yes)
+		(in_bom no)
 		(on_board yes)
 		(dnp no)
@@
 		(unit 1)
 		(exclude_from_sim no)
-		(in_bom yes)
+		(in_bom no)
 		(on_board yes)
 		(dnp no)
@@
 		(unit 1)
 		(exclude_from_sim no)
-		(in_bom yes)
+		(in_bom no)
 		(on_board yes)
 		(dnp no)
@@
 		(unit 1)
 		(exclude_from_sim no)
-		(in_bom yes)
+		(in_bom no)
 		(on_board yes)
 		(dnp no)
@@
 			)
 		)
-		(property "MFPN" "SBA0520Q or similar"
+		(property "MFPN" "RB161QS-40T18R"
 			(at 262.89 195.58 0)
 			(effects
@@
 			)
 		)
-		(property "LCSC" ""
+		(property "LCSC" "C2837790"
+			(at 262.89 195.58 0)
+			(effects
+				(font
+					(size 1.27 1.27)
+				)
+				(hide yes)
+			)
+		)
+		(property "VfVr" "20V"
+			(at 262.89 195.58 0)
+			(effects
+				(font
+					(size 1.27 1.27)
+				)
+				(hide yes)
+			)
+		)
+		(property "Rectified Current" "500mA"
 			(at 262.89 195.58 0)
 			(effects
@@
 			)
 		)
-		(property "MFPN" "SBA0520Q or similar"
+		(property "MFPN" "RB161QS-40T18R "
 			(at 186.69 137.16 0)
 			(effects
@@
 			)
 		)
-		(property "LCSC" ""
+		(property "LCSC" "C2837790"
 			(at 186.69 137.16 0)
 			(effects
@@
 		(unit 1)
 		(exclude_from_sim no)
-		(in_bom yes)
+		(in_bom no)
 		(on_board yes)
 		(dnp no)
@@
 			)
 		)
-		(property "Value" "74LVC1T45GM,115"
+		(property "Value" "74LVC1T45GM-Q100X"
 			(at 158.75 52.07 0)
 			(effects
@@
 			)
 		)
-		(property "LCSC" "C548481, C548480, C548479"
+		(property "LCSC" "C548481"
 			(at 158.75 59.69 0)
 			(effects
@@
 			)
 		)
-		(property "MFPN" "74LVC1T45GM,115"
+		(property "MFPN" "74LVC1T45GM-Q100X"
 			(at 158.75 59.69 0)
 			(effects
@@
 			)
 		)
+		(property "LCSC" "C76886"
+			(at 194.31 171.45 90)
+			(effects
+				(font
+					(size 1.27 1.27)
+				)
+				(hide yes)
+			)
+		)
 		(pin "1"
 		)
@@
 			)
 		)
-		(property "Value" "74LVC1T45GM,115"
+		(property "Value" "74LVC1T45GM-Q100X"
 			(at 158.75 35.56 0)
 			(effects
@@
 			)
 		)
-		(property "LCSC" "C548481, C548480, C548479"
+		(property "LCSC" "C548481"
 			(at 158.75 43.18 0)
 			(effects
@@
 			)
 		)
-		(property "MFPN" "74LVC1T45GM,115"
+		(property "MFPN" "74LVC1T45GM-Q100X"
 			(at 158.75 43.18 0)
 			(effects
@@
 		(unit 1)
 		(exclude_from_sim no)
-		(in_bom yes)
+		(in_bom no)
 		(on_board yes)
 		(dnp no)
@@
 			)
 		)
-		(property "Value" "74LVC1T45GM,115"
+		(property "Value" "74LVC1T45GM-Q100X"
 			(at 158.75 68.58 0)
 			(effects
@@
 			)
 		)
-		(property "LCSC" "C548481, C548480, C548479"
+		(property "LCSC" "C548481"
 			(at 158.75 76.2 0)
 			(effects
@@
 			)
 		)
-		(property "MFPN" "74LVC1T45GM,115"
+		(property "MFPN" "74LVC1T45GM-Q100X"
 			(at 158.75 76.2 0)
 			(effects
@@
 		(unit 1)
 		(exclude_from_sim no)
-		(in_bom yes)
+		(in_bom no)
 		(on_board yes)
 		(dnp no)
@@
 			)
 		)
-		(property "Value" "74LVC1T45GM,115"
+		(property "Value" "74LVC1T45GM-Q100X"
 			(at 158.75 19.05 0)
 			(effects
@@
 			)
 		)
-		(property "LCSC" "C548481, C548480, C548479"
+		(property "LCSC" "C548481"
 			(at 158.75 26.67 0)
 			(effects
@@
 			)
 		)
-		(property "MFPN" "74LVC1T45GM,115"
+		(property "MFPN" "74LVC1T45GM-Q100X"
 			(at 158.75 26.67 0)
 			(effects
@@
 			)
 		)
-		(property "Value" "74LVC1T45GM,115"
+		(property "Value" "74LVC1T45GM-Q100X"
 			(at 158.75 101.6 0)
 			(effects
@@
 			)
 		)
-		(property "LCSC" "C548481, C548480, C548479"
+		(property "LCSC" "C548481"
 			(at 158.75 109.22 0)
 			(effects
@@
 			)
 		)
-		(property "MFPN" "74LVC1T45GM,115"
+		(property "MFPN" "74LVC1T45GM-Q100X"
 			(at 158.75 109.22 0)
 			(effects
@@
 			)
 		)
-		(property "Value" "74LVC1T45GM,115"
+		(property "Value" "74LVC1T45GM-Q100X"
 			(at 158.75 85.09 0)
 			(effects
@@
 			)
 		)
-		(property "LCSC" "C548481, C548480, C548479"
+		(property "LCSC" "C548481"
 			(at 158.75 92.71 0)
 			(effects
@@
 			)
 		)
-		(property "MFPN" "74LVC1T45GM,115"
+		(property "MFPN" "74LVC1T45GM-Q100X"
 			(at 158.75 92.71 0)
 			(effects

Commit message: deleted all silkscreens and generated some gerbers
Parts:
- D1: MFPN LTST-C19HE1WT or ‎IN-S66TBTRGB‎ -> LTST-C19HE1WT or ‎IN-S66TBTRGB‎
- D2: MFPN RB161QS-40T18R -> RB161QS-40T18R
- R20: LCSC (none) -> C105872
Changed lines of the file:
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@@
 			)
 		)
-		(property "MFPN" "LTST-C19HE1WT or  ‎IN-S66TBTRGB‎"
+		(property "MFPN" "LTST-C19HE1WT or ‎IN-S66TBTRGB‎"
 			(at 138.43 270.51 0)
 			(effects
@@
 			)
 		)
+		(property "LCSC" "C105872"
+			(at 196.85 147.32 0)
+			(effects
+				(font
+					(size 1.27 1.27)
+				)
+				(hide yes)
+			)
+		)
 		(pin "1"
 		)
@@
 			)
 		)
-		(property "MFPN" "RB161QS-40T18R "
+		(property "MFPN" "RB161QS-40T18R"
 			(at 186.69 137.16 0)
 			(effects
